File: ePaper_timetable.kicad_sch (KiCad schematic)
At the start: 46 parts, among them J1 52435-2471, J2 Charging input - 5V, J3 Battery connector, Q1 BSS138, Q2 AO3401A, Q3 FS8205A, SW1 SW_Push, SW2 SW_Push, SW3 SW_Push, U1 Pico, U2 DW01A, U3 TP4056

Commit message: update sch and lib
Parts:
- removed U1: Pico, MCU_RaspberryPi_and_Boards:RPi_Pico_SMD_TH, symbol MCU_RaspberryPi_and_Boards:Pico
- added A1: RaspberryPi-Pico(W), MCU_RPi_Pico:Raspberry_Pi_Pico_W_SMT, symbol PicoW:RaspberryPi-Pico(W)
- added J4, J5, J6: Conn_01x03_Socket, symbol Connector:Conn_01x03_Socket
- added J7: USB_C_Receptacle_USB2.0, Connector_USB:USB_C_Receptacle_GCT_USB4105-xx-A_16P_TopMnt_Horizontal, symbol Connector:USB_C_Receptacle_USB2.0
- added R12, R13: 100R, Resistor_SMD:R_0805_2012Metric_Pad1.20x1.40mm_HandSolder, symbol Device:R
- added SW4, SW5: SW_Push, symbol Switch:SW_Push
- added U1: USBLC6-2P6, Package_SON:Texas_S-PWSON-N10, symbol Power_Protection:USBLC6-2P6
- added U4: USBLC6-2SC6, Package_TO_SOT_SMD:SOT-23-6, symbol Power_Protection:USBLC6-2SC6
- added U5: USBLC6-4SC6, Package_TO_SOT_SMD:SOT-23-6, symbol Power_Protection:USBLC6-4SC6
- D1, D2, D3: footprint Diode_SMD:D_0805_2012Metric_Pad1.15x1.40mm_HandSolder -> Diode_SMD:D_SOD-123
Connections:
- net 3.3V: now also A1.36 (3V3)
- net DW01_{Vcc}: now also SW5.1
- net EPD_BUSY': now also A1.17 (GPIO13)
- net EPD_CS': now also A1.12 (GPIO9)
- net EPD_DC': now also A1.11 (GPIO8)
- net EPD_DIN': now also A1.15 (GPIO11)
- net EPD_RST': now also A1.16 (GPIO12)
- net EPD_SCK': now also A1.14 (GPIO10)
- net GND: now also A1.13 (GND), A1.18 (GND), A1.23 (GND), A1.28 (GND), A1.3 (GND), A1.33 (AGND), A1.38 (GND), A1.42 (SWGND), A1.51 (TP6_BOOTSEL), A1.8 (GND), J4.2 (Pin_2), J5.2 (Pin_2), J6.2 (Pin_2), SW4.2
- net SW1: now also A1.24 (GPIO18)
- net SW2: now also A1.25 (GPIO19)
- net SW3: now also A1.26 (GPIO20)
- net at Q2.2 (S): now also A1.39 (VSYS)
- net at Q2.1 (G): now also A1.40 (VBUS)
- net at R8.1, U2.2 (CS): now also SW5.2
- new net: A1.30 (RUN), SW4.1
- new net: J4.1 (Pin_1), J5.1 (Pin_1), R12.1
- new net: J4.3 (Pin_3), J5.3 (Pin_3), R13.1
- new net: J7.A1 (GND), J7.A12 (GND), J7.B1 (GND), J7.B12 (GND)
- new net: J7.A4 (VBUS), J7.A9 (VBUS), J7.B4 (VBUS), J7.B9 (VBUS)
- new net BOOTSEL: A1.51 (TP6_BOOTSEL)
- new net SWCLK: A1.41 (SWCLK), R12.2
- new net SWDIO: A1.43 (SWDIO), R13.2
- new net UART0_RX: A1.2 (GPIO1), J6.1 (Pin_1)
- new net UART0_TX: A1.1 (GPIO0), J6.3 (Pin_3)
- new net USB_DM: A1.51 (TP6_BOOTSEL), J7.A7 (D-), J7.B7 (D-)
- new net USB_DP: A1.51 (TP6_BOOTSEL), J7.A6 (D+), J7.B6 (D+)
- no-connect marks 29 -> 19
Other:
- moved on the sheet: C14, J3, Q3, R8, R9, U2

Commit message: Update ePaper_timetable.kicad_sch
Parts:
- removed U1: USBLC6-2P6, Package_SON:Texas_S-PWSON-N10, symbol Power_Protection:USBLC6-2P6
- removed U5: USBLC6-4SC6, Package_TO_SOT_SMD:SOT-23-6, symbol Power_Protection:USBLC6-4SC6
- added F1: Polyfuse, symbol Device:Polyfuse
- added R14, R15: 100R, Resistor_SMD:R_0805_2012Metric_Pad1.20x1.40mm_HandSolder, symbol Device:R
- added R16, R17: 5k1, Resistor_SMD:R_0805_2012Metric_Pad1.20x1.40mm_HandSolder, symbol Device:R
Connections:
- net GND: now also J7.A1 (GND), J7.A12 (GND), J7.B1 (GND), J7.B12 (GND), J7.S1 (SHIELD), U4.2 (GND), R16.2, R17.2
- net UART0_RX: now also R14.2; no longer J6.1 (Pin_1)
- net UART0_TX: now also R15.2; no longer J6.3 (Pin_3)
- net USB_DM: now also U4.4 (I/O2); no longer J7.A7 (D-), J7.B7 (D-)
- net USB_DP: now also U4.3 (I/O2); no longer J7.A6 (D+), J7.B6 (D+)
- net I2C0_SDA: now reaches A1.6 (GPIO4)
- net I2C0_SCL: now reaches A1.7 (GPIO5)
- net at U4.1 (I/O1): now also J7.A6 (D+), J7.B6 (D+)
- net at U4.5 (VBUS): now also F1.2
- net at U4.6 (I/O1): now also J7.A7 (D-), J7.B7 (D-)
- net at J7.A4 (VBUS), J7.A9 (VBUS), J7.B4 (VBUS)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: now also F1.1
- net at J7.A5 (CC1): now also R16.1
- net at J7.B5 (CC2): now also R17.1
- new net: J6.3 (Pin_3), R15.1
- new net: J6.1 (Pin_1), R14.1
- no-connect marks 19 -> 23
Other:
- moved on the sheet: U4

Commit message: update sch and pcb
Parts:
- removed A1: RaspberryPi-Pico(W), MCU_RPi_Pico:Raspberry_Pi_Pico_W_SMT, symbol PicoW:RaspberryPi-Pico(W)
- added A1: RaspberryPi-Pico(W), MCU_RPi_Pico:Raspberry_Pi_Pico_W_SMT, symbol MCU_RPi_Pico:RaspberryPi-Pico(W)
- added C15: 1n, Capacitor_SMD:C_0805_2012Metric_Pad1.18x1.45mm_HandSolder, symbol Device:C
- added J7: Conn_01x04_Socket, Connector_PinSocket_2.54mm:PinSocket_1x04_P2.54mm_Vertical, symbol Connector:Conn_01x04_Socket
- added J9: Conn_01x01_Pin, Connector_Wire:SolderWirePad_1x01_SMD_1x2mm, symbol Connector:Conn_01x01_Pin
- added Q4: BSS138, Package_TO_SOT_SMD:SOT-23, symbol Transistor_FET:BSS138
- added R12, R15: 10k, Resistor_SMD:R_0805_2012Metric_Pad1.20x1.40mm_HandSolder, symbol Device:R
- added R16, R6: 0R, Resistor_SMD:R_1206_3216Metric_Pad1.30x1.75mm_HandSolder, symbol Device:R
- added R22: 200k, Resistor_SMD:R_0805_2012Metric_Pad1.20x1.40mm_HandSolder, symbol Device:R
- added R23: 100k, Resistor_SMD:R_0805_2012Metric_Pad1.20x1.40mm_HandSolder, symbol Device:R
- C1, C10, C11, C12, C2, C3, C4, C5, C6, C7, C8, C9: footprint Capacitor_SMD:C_1206_3216Metric_Pad1.33x1.80mm_HandSolder -> Capacitor_SMD:C_0805_2012Metric_Pad1.18x1.45mm_HandSolder
- C16: renamed from C15; footprint Capacitor_SMD:C_1206_3216Metric_Pad1.33x1.80mm_HandSolder -> Capacitor_SMD:C_0805_2012Metric_Pad1.18x1.45mm_HandSolder
- F1: footprint (none) -> Fuse:Fuse_1812_4532Metric_Pad1.30x3.40mm_HandSolder
- J3: renamed from J4; footprint (none) -> Connector_PinSocket_2.54mm:PinSocket_1x03_P2.54mm_Vertical
- J4: renamed from J2; footprint (none) -> Connector_Phoenix_MC:PhoenixContact_MC_1,5_2-G-3.81_1x02_P3.81mm_Horizontal
- J5: renamed from J6; footprint (none) -> Connector_PinSocket_2.54mm:PinSocket_1x03_P2.54mm_Vertical
- J6: renamed from J5; footprint (none) -> Connector_PinSocket_2.54mm:PinSocket_1x03_P2.54mm_Vertical
- J8: renamed from J3; footprint Connector_JST:JST_EH_S2B-EH_1x02_P2.50mm_Horizontal -> Connector_PinSocket_2.54mm:PinSocket_1x02_P2.54mm_Vertical
- SW1: renamed from SW4; footprint (none) -> Button_Switch_SMD:SW_Tactile_SPST_NO_Straight_CK_PTS636Sx25SMTRLFS
- SW5: footprint (none) -> Button_Switch_SMD:SW_Tactile_SPST_NO_Straight_CK_PTS636Sx25SMTRLFS
- U3: footprint Package_SO:HTSOP-8-1EP_3.9x4.9mm_P1.27mm_EP2.4x3.2mm_ThermalVias -> Package_SO:HTSOP-8-1EP_3.9x4.9mm_P1.27mm_EP2.4x3.2mm
- renumbered J7 to J1, J1 to J2, R12 to R10, R13 to R11, R14 to R13, R15 to R14, R7 to R17, R8 to R18, R9 to R19, R10 to R20, R11 to R21, R16 to R4, R17 to R5, R4 to R7, R5 to R8, R6 to R9, SW1 to SW2, SW2 to SW3, SW3 to SW4, U4 to U1
Connections:
- net BOOTSEL: now also A1.56 (TP6_BOOTSEL), J9.1 (Pin_1)
- net EPD_BUSY': now also A1.17 (GPIO13)
- net EPD_CS': now also A1.12 (GPIO9)
- net EPD_DC': now also A1.11 (GPIO8)
- net EPD_DIN': now also A1.15 (GPIO11)
- net EPD_RST': now also A1.16 (GPIO12)
- net EPD_SCK': now also A1.14 (GPIO10)
- net GND: now also A1.13 (GND), A1.18 (GND), A1.23 (GND), A1.28 (GND), A1.3 (GND), A1.33 (AGND), A1.38 (GND), A1.42 (SWGND), A1.51 (TP1_USB_GND), A1.8 (GND), C15.1, J7.4 (Pin_4), R23.2
- net I2C0_SCL: now also A1.7 (GPIO5), J7.3 (Pin_3), R12.1
- net I2C0_SDA: now also A1.6 (GPIO4), J7.2 (Pin_2), R15.1
- net SW1: now also A1.24 (GPIO18)
- net SW2: now also A1.25 (GPIO19)
- net SW3: now also A1.26 (GPIO20)
- net SWCLK: now also A1.41 (SWCLK)
- net SWDIO: now also A1.43 (SWDIO)
- net UART0_RX: now also A1.2 (GPIO1)
- net UART0_TX: now also A1.1 (GPIO0)
- net USB_DM: now also A1.52 (TP2_USB_DM)
- net USB_DP: now also A1.53 (TP3_USB_DP)
- net at SW1.1: now also A1.30 (RUN)
- net at Q2.2 (S): now also A1.39 (VSYS)
- net +5V: now reaches Q2.1 (G)
- net +5V: now also C13.2, D4.2 (A), D5.2 (A), U3.4 (VCC), U3.8 (CE), A1.40 (VBUS), R16.2, R6.2
- net BAT_CHRG: now reaches R21.2, U3.7 (~{CHRG})
- net BAT_CHRG: now also A1.5 (GPIO3)
- net BAT_STDBY: now reaches R20.2, U3.6 (~{STDBY})
- net BAT_STDBY: now also A1.4 (GPIO2)
- net at F1.2, U1.5 (VBUS): now also R6.1
- net 3.3V renamed +3V3
- net +3V3: now also A1.36 (3V3), J7.1 (Pin_1), Q4.1 (G), R12.2, R15.2
- net Battery- renamed -BATT
- net V_{battery} renamed +BATT
- net +BATT: now also R22.1
- new net: C15.2, Q4.3 (D), R22.2, R23.1
- new net: J4.2 (Pin_2), R16.1
- new net BAT_ADC: A1.34 (GPIO28_ADC2), Q4.2 (S)
- no-connect marks 23 -> 20
Other:
- moved on the sheet: F1, J1, J3, J5, J6, Q2, R10, R11, R13, R14, R4, R5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
