File: ePaper_timetable.kicad_pcb (KiCad board)
At the start: 2 copper layers, 95.2 x 80.6 mm, 72 parts, among them J1 USB_C_Receptacle_USB2.0, J2 Conn_01x01_Pin, J3 52435-2471, J4 Conn_01x03_Socket, J5 Charging input - 5V, J6 Conn_01x03_Socket, J7 Conn_01x03_Socket, J8 Conn_01x04_Socket, J9 Battery connector, Q1 BSS138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

Commit message: minor changes
Parts:
- added H1: MountingHole_Pad, MountingHole:MountingHole_3.2mm_M3_Pad, F.Cu at (71.1, 83.2)
- added H2: MountingHole_Pad, MountingHole:MountingHole_3.2mm_M3_Pad, F.Cu at (158.8, 83.2)
- added H3: MountingHole_Pad, MountingHole:MountingHole_3.2mm_M3_Pad, F.Cu at (71.1, 156.2)
- added H4: MountingHole_Pad, MountingHole:MountingHole_3.2mm_M3_Pad, F.Cu at (134.6, 142.2)
- added J10: Conn_01x01_Pin, Connector_Wire:SolderWirePad_1x01_SMD_1x2mm, F.Cu at (132.1, 118.7)
- added J11: Conn_01x01_Pin, Connector_Wire:SolderWirePad_1x01_SMD_1x2mm, F.Cu at (134.6, 118.7)
- added J12: Conn_01x01_Pin, Connector_Wire:SolderWirePad_1x01_SMD_1x2mm, F.Cu at (157.5, 118.7)
- added J13: Conn_01x01_Pin, Connector_Wire:SolderWirePad_1x01_SMD_1x2mm, F.Cu at (160.0, 118.7)
- J7: footprint Connector_PinSocket_2.54mm:PinSocket_1x03_P2.54mm_Vertical -> Connector_JST:JST_SH_BM03B-SRSS-TB_1x03-1MP_P1.00mm_Vertical
- moved J7 6.84 mm to (146.1, 82.5), turned to 0 degrees
- moved J4 5.46 mm to (143.5, 88.6)
- moved J9 3.03 mm to (94.0, 85.1), turned to -90 degrees
- moved J6 0.92 mm to (106.0, 120.0)
- moved J5 0.39 mm to (75.4, 111.7)
Connections:
- A1 pad 10: unconnected-(A1-GPIO7-Pad10) -> Net-(A1-GPIO7)
- A1 pad 19: unconnected-(A1-GPIO14-Pad19) -> Net-(A1-GPIO14)
- A1 pad 20: unconnected-(A1-GPIO15-Pad20) -> Net-(A1-GPIO15)
- A1 pad 9: unconnected-(A1-GPIO6-Pad9) -> Net-(A1-GPIO6)
- J3 pad 25: GND -> (no net)
- J9 pad 1: +BATT -> -BATT
- J9 pad 2: -BATT -> +BATT
Routing:
- net Net-(A1-GPIO7): track 0.00 -> 3.53 mm
- net Net-(A1-GPIO6): track 0.00 -> 3.53 mm
- net Net-(A1-GPIO15): track 0.00 -> 3.53 mm
- net Net-(A1-GPIO14): track 0.00 -> 3.53 mm
- net +BATT: track 48.9 -> 46.5 mm
- net -BATT: track 21.2 -> 19.8 mm
- net GND: track 0.65 -> 2.01 mm, vias 96 -> 161
- net +3V3: track 156.0 -> 154.9 mm
- net Net-(J6-Pin_1): track 3.73 -> 4.72 mm
- net Net-(F1-Pad1): track 11.7 -> 10.8 mm
- net Net-(J6-Pin_3): track 7.87 -> 8.49 mm
- net /EPD_BUSY': track 26.7 -> 26.2 mm
- net +5V: track 129.4 -> 130.0 mm
- net (no net): vias 4 -> 0
Other:
- outline, holes or cut-outs redrawn
- board text added: "+"
- board text added: "+5V"
- board text added: "-"
- board text added: "BAT"
- board text added: "DEBUG"
- board text added: "GND"
- board text added: "RX"
- board text added: "TX"
- board text added: "UART"
- board text added: "ePaper Timetable"

Commit message: gerbers generated
Parts:
- removed REF**: 7_5 inch display, 7_5 inch display model:7_5 inch display
